File: kicad/bbbmini/bbbmini.kicad_pcb (KiCad board)
At the start: 2 copper layers, 86.4 x 54.6 mm, 25 parts, among them P1 RC_OUTPUT, P10 GPS, P11 5V_INPUT, P12 SPI0, P13 CANBUS, P14 CANBUS R, P15 I2C2, P16 RC_1, P17 RC_3, P18 RC_4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

Commit message: Rev 1.4
Parts:
- added P19: HC_SR04, Pin_Headers:Pin_Header_Straight_1x04, F.Cu at (131.4, 119.4)
- added R2: 1k, Resistors_ThroughHole:Resistor_Horizontal_RM10mm, B.Cu at (151.9, 97.8)
- added R3: 2k, Resistors_ThroughHole:Resistor_Horizontal_RM10mm, B.Cu at (149.0, 97.8)
- added R4: 1k, Resistors_ThroughHole:Resistor_Horizontal_RM10mm, B.Cu at (143.1, 97.8)
- added R5: 2k, Resistors_ThroughHole:Resistor_Horizontal_RM10mm, B.Cu at (146.1, 97.8)
- P10: footprint Pin_Headers:Pin_Header_Straight_1x04 -> Pin_Headers:Pin_Header_Straight_1x05
- P4: value RC INPUT -> RC_IN; footprint Pin_Headers:Pin_Header_Straight_1x03 -> Pin_Headers:Pin_Header_Straight_1x04
- U1: footprint Housings_DIP:DIP-8__300 -> Housings_DIP:DIP-8_W7.62mm
- moved P3 52.5 mm to (137.2, 92.7)
- moved P15 10.8 mm to (146.7, 119.4)
- moved P7 8.89 mm to (161.9, 119.4)
- moved P12 6.99 mm to (182.2, 119.4)
- moved U1 4.96 mm to (156.8, 92.7), turned to 90 degrees
- moved P4 4.07 mm to (137.2, 85.1), turned to 270 degrees
- moved P17 2.41 mm to (114.7, 114.3)
- moved P11 1.91 mm to (123.8, 125.1)
- moved P6 1.91 mm to (167.0, 110.5)
- moved REF3 1.91 mm to (181.0, 101.5)
- moved P5 1.27 mm to (136.5, 110.5)
- moved REF1 1.27 mm to (137.8, 98.8)
- moved REF2 1.27 mm to (158.2, 98.8)
- moved P10 1.05 mm to (151.9, 85.1)
- moved C1 1.02 mm to (171.2, 85.1)
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Connections:
- net / SPI1_SCLK renamed /SPI1_SCLK
- net /MPU9250_CS renamed /SPI1_CS0
- net /MS5611_CS renamed /SPI1_CS1
- P10 pad 1: GND -> +5V
- P10 pad 3: /GPS_RX -> GND
- P10 pad 4: /GPS_TX -> /GPS_RX
- P4 pad 1: +3V3 -> +5V
- P4 pad 2: GND -> +3V3
- P4 pad 3: /RC_IN -> GND
- P5 pad 8: Net-(P5-Pad8) -> /MPU9250_INT
- P8 pad 12: Net-(P8-Pad12) -> /SR04_TRIG
- P8 pad 16: Net-(P8-Pad16) -> /SR04_ECHO
- P9 pad 25: Net-(P9-Pad25) -> /MPU9250_INT
Routing:
- net /SR04_TRIG: track 0.00 -> 59.4 mm
- net Net-(P2-Pad10): track 40.5 -> 95.2 mm
- net +5V: track 109.0 -> 152.5 mm
- net Net-(P19-Pad3): track 0.00 -> 37.3 mm
- net GND: track 270.6 -> 300.9 mm
- net /I2C2_SCL: track 42.4 -> 19.9 mm
- net /MPU9250_INT: track 0.00 -> 22.4 mm
- net Net-(P4-Pad4): track 0.00 -> 20.7 mm
- net /SR04_ECHO: track 0.00 -> 17.3 mm
- net /SPI1_MISO: track 54.2 -> 70.8 mm
- net /RC_IN: track 13.8 -> 30.4 mm
- net /RC_4: track 72.8 -> 59.3 mm
- net /RC_2: track 49.9 -> 63.1 mm
- net +3V3: track 149.8 -> 161.3 mm, vias 0 -> 1
- net /CAN_TX: track 48.0 -> 37.2 mm, vias 1 -> 0
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- added copper zone on B.Cu, net GND
- added copper zone on F.Cu, net GND
Other:
- board text added: "3.3V"
- board text added: "5V"
- board text added: "5V IN"
- board text added: "BBBMINI Rev. 1.4"
- board text added: "ECHO"
- board text added: "GPS/UART5"
- board text added: "HC-SR04"
- board text added: "I/O PINS 3.3V!"
- board text added: "INT"
- board text added: "RCIN"
- board text added: "TRIG"
- board text added: "Telemetry/UART4"
- board text added: "by Mirko Denecke"
- board text removed: "+3V3"
- board text removed: "+5V"
- board text removed: "+5V IN"
- board text removed: "5V Input"
- board text removed: "5V to RC_X"
- board text removed: "ALL I/O PINS 3.3V!"
- board text removed: "BBBMINI Rev. 1.2"
- board text removed: "CAN_R"
- board text removed: "GPS / UART5"
- board text removed: "RC_IN"
- board text removed: "Telemetry / UART4"

Commit message: Rev. 1.5
Parts:
- added P20: I2C2, Pin_Headers:Pin_Header_Straight_1x05, F.Cu at (131.4, 115.8)
- added P21: V / I, Pin_Headers:Pin_Header_Straight_1x03, F.Cu at (182.2, 92.7)
- added R6: 20k, Resistors_ThroughHole:Resistor_Horizontal_RM10mm, B.Cu at (164.5, 101.1)
- added R7: 10k, Resistors_ThroughHole:Resistor_Horizontal_RM10mm, B.Cu at (167.0, 101.1)
- added R8: 20k, Resistors_ThroughHole:Resistor_Horizontal_RM10mm, B.Cu at (169.5, 101.1)
- added R9: 10k, Resistors_ThroughHole:Resistor_Horizontal_RM10mm, B.Cu at (172.1, 101.1)
- added REF**: Symbol_OSHW-Logo_SilkScreen, Symbols:Symbol_OSHW-Logo_SilkScreen, F.Cu at (125.3, 78.8)
- P3: value 5V FROM RC_OUT -> 5V TO RC_OUT
- R1: moved to B.Cu
- moved P3 45.3 mm to (182.2, 87.6), turned to 180 degrees
- moved R1 16.8 mm to (174.6, 101.1), turned to 90 degrees
- moved P15 15.2 mm to (131.4, 119.4)
- moved P19 12.7 mm to (144.1, 119.4)
- moved C1 5.70 mm to (168.7, 90.2), turned to 270 degrees
- moved C2 5.70 mm to (168.7, 87.6), turned to 90 degrees
- moved P14 5.67 mm to (177.1, 87.6)
- moved P13 5.23 mm to (179.7, 87.6)
- moved P7 2.54 mm to (159.4, 119.4)
- moved R4 1.02 mm to (144.1, 97.8)
- moved P16 0.64 mm to (120.4, 80.0)
- moved P4 0.63 mm to (136.5, 85.1)
- moved R5 0.63 mm to (146.7, 97.8)
- moved R3 0.25 mm to (149.2, 97.8)
- moved P10 0.13 mm to (151.8, 85.1)
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Connections:
- P9 pad 34: Net-(P9-Pad34) -> GND
- P9 pad 39: Net-(P9-Pad39) -> /VOLTAGE
- P9 pad 40: Net-(P9-Pad40) -> /CURRENT
- R3 pad 1: GND -> /SR04_ECHO
- R3 pad 2: Net-(P19-Pad3) -> GND
Routing:
- net Net-(P2-Pad10): track 95.2 -> 39.5 mm
- net /RC_3: track 132.5 -> 182.9 mm
- net /CURRENT: track 0.00 -> 35.2 mm
- net /VOLTAGE: track 0.00 -> 31.8 mm, vias 0 -> 1
- net /I2C2_SCL: track 19.9 -> 46.6 mm
- net GND: track 300.9 -> 324.2 mm
- net Net-(P21-Pad1): track 0.00 -> 23.2 mm
- net +5V: track 152.5 -> 173.7 mm, vias 0 -> 1
- net Net-(P14-Pad2): track 5.08 -> 23.6 mm, vias 0 -> 1
- net Net-(P21-Pad2): track 0.00 -> 17.8 mm
- net /I2C2_SDA: track 28.9 -> 43.9 mm
- net /SR04_TRIG: track 59.4 -> 45.2 mm
- net /SPI1_CS0: track 21.1 -> 35.2 mm
- net /CAN_RX: track 38.4 -> 49.6 mm
- net /RC_2: track 63.1 -> 52.5 mm
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Other:
- net class Default: trace_width 0.254 -> 0.3; via_dia 0.6604 -> 0.7
- net class power: via_dia 0.9144 -> 1.2
- board text added: "BBBMINI Rev. 1.5"
- board text added: "CUR"
- board text added: "R1 = 120Ω"
- board text added: "R2 = 1kΩ R3 = 2kΩ"
- board text added: "R6 & R8 = 20kΩ R7 & R9 = 10kΩ"
- board text added: "RCIN 3.3V → R4 = 0Ω R5 = not used RCIN 5.0V → R4 = 1kΩ R5 = 2kΩ"
- board text added: "VOL"
- board text added: "https://github.com/mirkix/BBBMINI"
- board text removed: "BBBMINI Rev. 1.4"
- board text removed: "I/O PINS 3.3V!"
